File: MidiToCV.kicad_pcb (KiCad board)
At the start: 2 copper layers, 150 x 80 mm, 67 parts, among them IC1 AD5724RBREZ, IC2 AD5724RBREZ, IC3 AD5724RBREZ, IC4 AD5724RBREZ, J1 AudioJack2_Ground_SwitchT, J10 AudioJack2_Ground_SwitchT, J11 AudioJack2_Ground_SwitchT, J12 AudioJack2_Ground_SwitchT, J13 AudioJack2_Ground_SwitchT, J14 AudioJack2_Ground_SwitchT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

Commit message: ladc_ bug fix
Parts:
- J10, J14, J2, J6: footprint MidiToCV:ACJS-NV35-XX -> ACJS-NV35-XX
Connections:
- IC2 pad 10: /sheet5FC111E9/_LDAC -> /Sheet5FA40E10/_LDAC
- IC3 pad 10: /sheet5FC111E9/_LDAC -> /Sheet5FA40E10/_LDAC
- IC4 pad 10: /sheet5FC111E9/_LDAC -> /Sheet5FA40E10/_LDAC
- J17 pad 7: /sheet5FC111E9/_LDAC -> /Sheet5FA40E10/_LDAC
- J17 pad 8: /sheet5FC111E9/_LDAC -> /Sheet5FA40E10/_LDAC
Routing:
- net /sheet5FC111E9/_LDAC: track 67.0 -> 0.00 mm, vias 2 -> 0
- net /Sheet5FA40E10/_LDAC: track 74.8 -> 118.6 mm, vias 0 -> 5
- net /Sheet5FA40E10/2.5Vref: track 90.0 -> 94.4 mm
- net /Sheet5FA40E10/SCLK: track 113.5 -> 110.4 mm
